File: hardware/ORGNET.kicad_pcb (KiCad board)
At the start: 2 copper layers, 21 x 50 mm, 41 parts, among them J1 Conn_02x08_Odd_Even, J3 Conn_01x03, U1 SN74LVC8T245, U2 SN74LVC8T245, U3 AP2112K-3.3, U4 RP2350A, U5 W25Q128JVP, U6 Raspberry Pi Radio Module 2, Y1 12M

Commit message: Add notch and use 0406 resistors/capacitors
Parts:
- C1, C10, C11, C12, C13, C14, C15, C16, C17, C18, C19, C2, C3, C4, C5, C6, C7, C8, C9: footprint Capacitor_SMD:C_0201_0603Metric_Pad0.64x0.40mm_HandSolder -> Capacitor_SMD:C_0402_1005Metric_Pad0.74x0.62mm_HandSolder
- R1, R2, R3, R4, R5, R6, R7, R8: footprint Resistor_SMD:R_0201_0603Metric_Pad0.64x0.40mm_HandSolder -> Resistor_SMD:R_0402_1005Metric_Pad0.72x0.64mm_HandSolder
- moved C12 4.39 mm to (157.3, 93.2), turned to -90 degrees
- moved R4 3.04 mm to (161.1, 92.0), turned to 180 degrees
- moved C15 2.52 mm to (161.2, 90.8), turned to 0 degrees
- moved C14 2.09 mm to (159.4, 92.5)
- moved C13 1.64 mm to (158.3, 93.2)
- moved R1 1.13 mm to (147.6, 100.7)
- moved R6 0.75 mm to (145.8, 100.2), turned to -90 degrees
- moved R3 0.46 mm to (161.5, 100.8)
- moved C10 0.40 mm to (159.3, 98.4)
- moved C11 0.39 mm to (159.3, 99.4)
- moved C1 0.38 mm to (145.3, 106.8)
- moved C4 0.36 mm to (161.5, 99.8)
- moved C8 0.31 mm to (143.5, 100.7)
- moved C18 0.28 mm to (161.5, 98.8)
- moved R8 0.23 mm to (157.6, 91.5)
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Connections:
- U4 pad 7: unconnected-(U4-GPIO4-Pad7) -> RP_SCLK
- U4 pad 8: RP_SCLK -> unconnected-(U4-GPIO5-Pad8)
Routing:
- net SVCC: track 49.1 -> 41.4 mm
- net +3V3: track 116.9 -> 123.9 mm
- net GND: track 35.2 -> 40.3 mm, vias 31 -> 29
- net RP_SD7: track 4.62 -> 3.88 mm
- net Net-(U4-RUN): track 5.82 -> 6.29 mm, vias 1 -> 2
Other:
- outline, holes or cut-outs redrawn
